File: kicad/tta8_lsu/tta8_lsu.kicad_pcb (KiCad board)
At the start: 2 copper layers, 92 x 100 mm, 15 parts, among them J1 Conn_02x32_Counter_Clockwise, J2 Conn_01x06, J3 Conn_02x02_Odd_Even, U1 74AHCT573, U2 74AHCT573, U3 74AHCT573, U4 74AHCT573, U5 74AHCT573, U6 74AHCT573, U7 74AHCT00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

Commit message: Ground fill changes + gerber zip
Routing:
- net +5V: track 283.4 -> 284.1 mm
Changed lines of the file:
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@@
 	)
 	(segment
-		(start 102.4 127.9)
+		(start 109 133.3)
 		(end 109 134.5)
 		(width 0.5)
@@
 	)
 	(segment
+		(start 101.7 127.9)
+		(end 104.6 130.8)
+		(width 0.5)
+		(layer "B.Cu")
+		(net 66)
+	)
+	(segment
 		(start 90.635 127.9)
-		(end 102.4 127.9)
+		(end 101.7 127.9)
 		(width 0.5)
 		(layer "B.Cu")
@@
 		(width 0.5)
 		(layer "B.Cu")
+		(net 66)
+	)
+	(segment
+		(start 106.5 130.8)
+		(end 109 133.3)
+		(width 0.5)
+		(layer "B.Cu")
+		(net 66)
+	)
+	(segment
+		(start 104.6 130.8)
+		(end 106.5 130.8)
+		(width 0.5)
+		(layer "B.Cu")

Commit message: Fix second address pointer register
Was T->A supposed to be T->T
Connections:
- U3 pad 12: A8 -> T8
- U3 pad 13: A9 -> T9
- U3 pad 14: A10 -> T10
- U3 pad 15: A11 -> T11
- U3 pad 16: A12 -> T12
- U3 pad 17: A13 -> T13
- U3 pad 18: A14 -> T14
- U3 pad 19: A15 -> T15
- U4 pad 12: A0 -> T0
- U4 pad 13: A1 -> T1
- U4 pad 14: A2 -> T2
- U4 pad 15: A3 -> T3
- U4 pad 16: A4 -> T4
- U4 pad 17: A5 -> T5
- U4 pad 18: A6 -> T6
- U4 pad 19: A7 -> T7
Routing:
- net Net-(U1-OE): track 119.6 -> 86.0 mm, vias 3 -> 2
- net A11: track 52.6 -> 33.4 mm
- net A9: track 53.0 -> 33.9 mm
- net A14: track 52.5 -> 33.4 mm
- net A12: track 52.5 -> 33.5 mm
- net A10: track 52.5 -> 33.5 mm
- net A15: track 52.5 -> 33.4 mm
- net A13: track 52.4 -> 33.4 mm
- net A8: track 52.5 -> 33.4 mm
- net A2: track 44.2 -> 25.2 mm
- net A5: track 42.8 -> 23.8 mm
- net A0: track 44.2 -> 25.2 mm
- net A3: track 44.2 -> 25.2 mm
- net A6: track 42.6 -> 23.7 mm
- net A1: track 44.2 -> 25.2 mm
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
Commit message: Add decoupling to tt8 lsu
Parts:
- added C1: 0.1uF, Capacitor_THT:C_Disc_D5.0mm_W2.5mm_P2.50mm, F.Cu at (72.7, 128.7)
- added C2: 0.1uF, Capacitor_THT:C_Disc_D5.0mm_W2.5mm_P2.50mm, F.Cu at (72.7, 98.6)
- added C3: 0.1uF, Capacitor_THT:C_Disc_D5.0mm_W2.5mm_P2.50mm, F.Cu at (90.8, 128.7)
- added C4: 0.1uF, Capacitor_THT:C_Disc_D5.0mm_W2.5mm_P2.50mm, F.Cu at (90.6, 98.6)
- added C5: 0.1uF, Capacitor_THT:C_Disc_D5.0mm_W2.5mm_P2.50mm, F.Cu at (102.3, 97.7)
- added C6: 0.1uF, Capacitor_THT:C_Disc_D5.0mm_W2.5mm_P2.50mm, F.Cu at (115.5, 97.6)
- added C7: 0.1uF, Capacitor_THT:C_Disc_D5.0mm_W2.5mm_P2.50mm, F.Cu at (68.3, 55.6)
- added C8: 0.1uF, Capacitor_THT:C_Disc_D5.0mm_W2.5mm_P2.50mm, F.Cu at (90.3, 55.8)
Routing:
- net +5V: track 283.6 -> 300.7 mm
- net D2: track 153.3 -> 156.2 mm
- net D0: track 173.9 -> 176.8 mm
- net D6: track 114.1 -> 117.0 mm
- net D3: track 143.6 -> 146.5 mm
- net D1: track 163.0 -> 165.9 mm
- net D5: track 123.9 -> 126.8 mm
- net D7: track 105.0 -> 108.0 mm
- net D4: track 133.6 -> 136.5 mm
- net T7: track 85.6 -> 88.1 mm
- net T6: track 91.4 -> 93.8 mm
- net T5: track 97.2 -> 99.7 mm
- net T4: track 102.8 -> 105.3 mm
- net T3: track 108.5 -> 111.0 mm
- net T2: track 114.4 -> 116.9 mm
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
Commit message: cu change to sockets
Changed lines of the file:
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@@
+	)
+	(segment
+		(start 73.4 121.04)
+		(end 73.4 105.7)
+		(width 0.2)
+		(layer "F.Cu")
+		(net 73)
 	)
 	(segment
@@
 	)
 	(segment
-		(start 73.4 105.7)
-		(end 73.4 121.04)
-		(width 0.2)
-		(layer "F.Cu")
-		(net 73)
-	)
-	(segment
 		(start 92.3 69.4)
 		(end 100.98 60.72)
@@
 	)
 	(segment
-		(start 73.4 121.04)
-		(end 77.72 125.36)
+		(start 77.72 125.36)
+		(end 73.4 121.04)
 		(width 0.2)
 		(layer "F.Cu")
